File: schematics/MotorController.sch (EAGLE design)
At the start: 30 parts, among them K1 35701331

Commit message: no message
Parts:
- removed POWER-INPUT: 1, con-lstb:MA03-1
- added DC_MOTOR_DRIVER: SINGLE_MOTOR_DRIVER, pololu motor driver:SINGLE_MOTOR_DRIVER
- added IC1: (no value), v-reg:78XXL
- added LED1: (no value), led:LED3MM
- added LOG-UART: 1, con-lstb:MA03-1
- added POWER_IN: (no value), SparkFun-Connectors:CONN_023.5MM
- added R11: 1K, resistor:R-EU_0204/5
- D1: value 1N4148DO35-7 -> 1N5400; device diode:1N4148DO35-7 -> diode:1N5400
- MOTOR1, MOTOR2, MOTOR3: value 1 -> 5566-4; device con-lstb:MA03-1 -> con-molex:5566-4
Connections:
- removed net GND: C1.-, C2.-, C3.2, CONTROL-I2C.3, DC-MOTOR.4, DRK1.GND, DRK2.GND, DRK3.GND, ENCODER1.4, ENCODER2.4, ENCODER3.4, IMU-I2C.3, POWER-INPUT.1, PRJ1.GND, T1.E
- removed net VCC: C1.+, C3.1, D1.C, DC-MOTOR.3, ENCODER1.1, ENCODER2.1, ENCODER3.1, K11.3, PRJ1.VIN
- new net BLCK-M2: DC-MOTOR.2, DC_MOTOR_DRIVER.OUT1
- new net ENC_B: DC-MOTOR.6, PRJ1.35/A16
- new net ENC_GND: C1.-, C2.-, C3.2, CONTROL-I2C.3, DC-MOTOR.3, DC_MOTOR_DRIVER.GND, DRK1.GND, DRK2.GND, DRK3.GND, ENCODER1.4, ENCODER2.4, ENCODER3.4, IC1.GND, IMU-I2C.3, LED1.A, LOG-UART.3, POWER_IN.1, PRJ1.GND, T1.E
- new net ENC_VCC: C1.+, C3.1, DC-MOTOR.4, DC_MOTOR_DRIVER.VDD(+5V), ENCODER1.1, ENCODER2.1, ENCODER3.1, IC1.OUT, K11.3, PRJ1.VIN, R11.2
- new net N$44: DC_MOTOR_DRIVER.IN1, PRJ1.29
- new net N$45: DC_MOTOR_DRIVER.EN, PRJ1.31/A12
- new net N$46: PRJ1.36/A17
- new net N$47: DC_MOTOR_DRIVER.IN2, PRJ1.30
- new net RED-M1: DC-MOTOR.1, DC_MOTOR_DRIVER.OUT2
- new net RX5: LOG-UART.1, PRJ1.34/A15
- new net TX5: LOG-UART.2, PRJ1.33/A14
- net N$1: now also MOTOR1-3.S; no longer MOTOR1.3
- net N$12: now also DC_MOTOR_DRIVER.VIN(5-28V)
- net N$13: now also MOTOR2-3.S; no longer MOTOR2.3
- net N$14: now also MOTOR2-2.S; no longer MOTOR2.2
- net N$15: now also MOTOR2-1.S; no longer MOTOR2.1
- net N$16: now also MOTOR3-3.S; no longer MOTOR3.3
- net N$17: now also MOTOR3-2.S; no longer MOTOR3.2
- net N$18: now also MOTOR3-1.S; no longer MOTOR3.1
- net N$2: now also MOTOR1-2.S; no longer MOTOR1.2
- net N$3: now also MOTOR1-1.S; no longer MOTOR1.1
- net N$32: now also D1.A, IC1.IN, POWER_IN.2; no longer K12.S, POWER-INPUT.3
- net N$39: now also D1.C, K12.S; no longer D1.A, POWER-INPUT.2
- net N$40: now also LED1.C, R11.1; no longer DC-MOTOR.2, PRJ1.33/A14
- net N$41: now also DC_MOTOR_DRIVER.INV, PRJ1.32/A13; no longer DC-MOTOR.1, PRJ1.34/A15
Other:
- moved on the sheet: C2, CONTROL-I2C, DC-MOTOR, IMU-I2C

Commit message: beltdrive wheels got a flange
Parts:
- added D2: 1N4148DO35-7, diode:1N4148DO35-7
- C1, C2: value (none) -> 470uF
- C3: value (none) -> 100nF
- IC1: value (none) -> 7805
- LED1: value (none) -> green
- POWER_IN: value (none) -> 12V
- T1: value (none) -> BC338
Connections:
- net ENC_B renamed WH_ENC_B
- net ENC_GND renamed GND
- removed net ENC_VCC: C1.+, C3.1, DC-MOTOR.4, DC_MOTOR_DRIVER.VDD(+5V), ENCODER1.1, ENCODER2.1, ENCODER3.1, IC1.OUT, K11.3, PRJ1.VIN, R11.2
- removed net N$46: PRJ1.36/A17
- new net VCC: C1.+, C3.1, D2.C, DC-MOTOR.4, DC_MOTOR_DRIVER.VDD(+5V), ENCODER1.1, ENCODER2.1, ENCODER3.1, IC1.OUT, K11.3, PRJ1.VIN, R11.2
- new net Y_ENC_A: DC-MOTOR.5, PRJ1.36/A17
- net N$31: now also D2.A

Commit message: no message
Parts:
- removed LED1: green, led:LED3MM
- removed R11: 1K, resistor:R-EU_0204/5
- removed T1: BC338, transistor:-NPN-TO92
- added Q1: BC307, transistor-pnp:BC307
- added SV1: (no value), con-lstb:MA04-1
- IMU-I2C: device con-lstb:MA03-1 -> con-lstb:MA05-1
Connections:
- removed net N$40: LED1.C, R11.1
- new net N$46: IMU-I2C.4, PRJ1.3V3_LO
- new net N$48: IMU-I2C.1, PRJ1.20/A6
- new net N$49: PRJ1.23/A9, SV1.1
- new net N$50: PRJ1.22/A8, SV1.2
- new net N$51: PRJ1.21/A7, SV1.3
- net GND: now also D2.A, IMU-I2C.5, K11.5, SV1.4; no longer IMU-I2C.3, LED1.A, T1.E
- net IMU-SCL: now also IMU-I2C.2; no longer IMU-I2C.1
- net IMU-SDA: now also IMU-I2C.3; no longer IMU-I2C.2
- net N$30: now also Q1.B; no longer T1.B
- net N$31: now also D2.C, K11.3, Q1.C; no longer D2.A, K11.5, T1.C
- net VCC: now also Q1.E; no longer D2.C, K11.3, R11.2
Other:
- moved on the sheet: D2, K1

Commit message: no message
Parts:
- removed DC_MOTOR_DRIVER: SINGLE_MOTOR_DRIVER, pololu motor driver:SINGLE_MOTOR_DRIVER
- removed K1: 35701331, relay:35701331
- added R11: 0, resistor:R-EU_0204/2V
- added REL1: HF49FD, relay:HF49FD
- added S1: (no value), switch-dil:DA02
- added U$1: SINGLE_MOTOR_DRIVER, pololu motor driver:SINGLE_MOTOR_DRIVER
Connections:
- new net LIPO-GND: DRK1.GND, DRK2.GND, DRK3.GND, POWER_IN.1, R11.1, U$1.GND
- new net LIPO-VDD: DRK1.LIPO+, DRK2.LIPO+, DRK3.LIPO+, REL1G$1.P, U$1.VIN(5-28V)
- new net N$40: PRJ1.39/A20, S1.4
- net BLCK-M2: now also U$1.OUT2; no longer DC_MOTOR_DRIVER.OUT1
- net GND: now also R11.2, REL1G$2.-, S1.1, S1.2; no longer DC_MOTOR_DRIVER.GND, DRK1.GND, DRK2.GND, DRK3.GND, K11.5, POWER_IN.1
- net N$12: now also PRJ1.A21/DAC0, S1.3; no longer DC_MOTOR_DRIVER.VIN(5-28V), DRK1.LIPO+, DRK2.LIPO+, DRK3.LIPO+, K12.P
- net N$31: now also REL1G$2.+; no longer K11.3
- net N$39: now also REL1G$1.S; no longer K12.S
- net N$41: now also U$1.INV; no longer DC_MOTOR_DRIVER.INV
- net N$44: now also U$1.IN1; no longer DC_MOTOR_DRIVER.IN1
- net N$45: now also U$1.EN; no longer DC_MOTOR_DRIVER.EN
- net N$47: now also U$1.IN2; no longer DC_MOTOR_DRIVER.IN2
- net RED-M1: now also U$1.OUT1; no longer DC_MOTOR_DRIVER.OUT2
- net VCC: now also U$1.VDD(+5V); no longer DC_MOTOR_DRIVER.VDD(+5V)
Other:
- moved on the sheet: CONTROL-I2C, DC-MOTOR

Commit message: no message
Connections:
- net N$10: now also PRJ1.24
- net N$21: now also PRJ1.5; no longer PRJ1.3/CANTX
- net N$22: now also PRJ1.6; no longer PRJ1.4/CANRX
- net N$23: now also PRJ1.7; no longer PRJ1.5
- net N$27: now also PRJ1.8; no longer PRJ1.6
- net N$28: now also PRJ1.9/CS; no longer PRJ1.7
- net N$29: now also PRJ1.10/CS; no longer PRJ1.8
- net N$33: now also ENCODER1.3, PRJ1.11/MOSI; no longer ENCODER3.3, PRJ1.9/CS
- net N$34: now also ENCODER1.2, PRJ1.12/MISO; no longer ENCODER3.2, PRJ1.10/CS
- net N$35: now also PRJ1.25; no longer PRJ1.11/MOSI
- net N$36: now also PRJ1.26; no longer PRJ1.12/MISO
- net N$37: now also ENCODER3.3, PRJ1.27; no longer ENCODER1.3, PRJ1.3V3
- net N$38: now also ENCODER3.2, PRJ1.28; no longer ENCODER1.2, PRJ1.24
- net N$42: no longer PRJ1.25
- net N$7: now also PRJ1.4/CANRX; no longer PRJ1.2
- net N$8: now also PRJ1.3/CANTX; no longer PRJ1.1/TX
- net N$9: now also PRJ1.2; no longer PRJ1.0/RX
Other:
- moved on the sheet: ENCODER1, ENCODER3
