File: schematics/MotorController.sch (EAGLE design)
At the start: 37 parts, among them IC1 7805, Q1 BC307

Commit message: no message
Parts:
- added HE1, HE2, HE3: 5566-6, con-molex:5566-6
- added S2: (no value), switch-omron:10-XX
Connections:
- new net N$52: PRJ1.RESET, S2.P
- new net N$53: HE1-5.S, HE2-5.S, HE3-5.S
- new net N$54: HE1-1.S, PRJ1.17/A3
- new net N$55: HE2-1.S, PRJ1.16/A2
- new net N$56: HE3-1.S, PRJ1.15/A1
- net GND: now also HE1-4.S, HE2-4.S, HE3-4.S, S2.S, S2.S1
- net N$42: now also PRJ1.0/RX

Commit message: First print of bottom sphere
Parts:
- removed SV1: (no value), con-lstb:MA04-1
Connections:
- new net N$57: HE1-2.S, PRJ1.1/TX
- new net N$58: HE1-3.S, PRJ1.14/A0
- new net N$59: HE2-3.S, PRJ1.13/SCK
- net GND: no longer SV1.4
- net N$49: now also HE3-2.S; no longer SV1.1
- net N$50: now also HE3-3.S; no longer SV1.2
- net N$51: now also HE2-2.S; no longer SV1.3
Other:
- moved on the sheet: IMU-I2C
Changed lines of the file:
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@@
 <part name="POWER_IN" library="SparkFun-Connectors" library_urn="urn:adsk.eagle:library:513" deviceset="CONN_02" device="3.5MM" package3d_urn="urn:adsk.eagle:package:38050/1" value="12V"/>
 <part name="D2" library="diode" library_urn="urn:adsk.eagle:library:210" deviceset="1N4148" device="DO35-7" package3d_urn="urn:adsk.eagle:package:43339/1"/>
-<part name="SV1" library="con-lstb" library_urn="urn:adsk.eagle:library:162" deviceset="MA04-1" device="" package3d_urn="urn:adsk.eagle:package:8337/1"/>
 <part name="Q1" library="transistor-pnp" library_urn="urn:adsk.eagle:library:399" deviceset="BC307" device="" package3d_urn="urn:adsk.eagle:package:29211/2"/>
 <part name="R11" library="resistor" library_urn="urn:adsk.eagle:library:348" deviceset="R-EU_" device="0204/2V" package3d_urn="urn:adsk.eagle:package:23495/1" value="0"/>
@@
 <instance part="ENCODER1" gate="1" x="190.5" y="50.8" rot="R180"/>
 <instance part="ENCODER2" gate="1" x="190.5" y="71.12" rot="R180"/>
-<instance part="IMU-I2C" gate="G$1" x="48.26" y="142.24" rot="R270"/>
+<instance part="IMU-I2C" gate="G$1" x="48.26" y="170.18" rot="R270"/>
 <instance part="CONTROL-I2C" gate="G$1" x="71.12" y="142.24" rot="R270"/>
 <instance part="DC-MOTOR" gate="1" x="254" y="132.08" rot="R180"/>
@@
 <instance part="POWER_IN" gate="G$1" x="-142.24" y="55.88"/>
 <instance part="D2" gate="G$1" x="-45.72" y="-12.7" rot="R90"/>
-<instance part="SV1" gate="1" x="40.64" y="160.02" rot="R270"/>
 <instance part="Q1" gate="G$1" x="-58.42" y="7.62"/>
 <instance part="R11" gate="G$1" x="-121.92" y="-30.48" rot="R90"/>
@@
 <wire x1="175.26" y1="48.26" x2="175.26" y2="-22.86" width="0.1524" layer="91"/>
 <junction x="175.26" y="48.26"/>
-<wire x1="53.34" y1="124.46" x2="58.42" y2="124.46" width="0.1524" layer="91"/>
-<wire x1="58.42" y1="124.46" x2="73.66" y2="124.46" width="0.1524" layer="91"/>
+<wire x1="53.34" y1="124.46" x2="73.66" y2="124.46" width="0.1524" layer="91"/>
 <wire x1="53.34" y1="124.46" x2="17.78" y2="124.46" width="0.1524" layer="91"/>
 <wire x1="17.78" y1="124.46" x2="15.24" y2="124.46" width="0.1524" layer="91"/>
@@
 <junction x="-109.22" y="-22.86"/>
 <pinref part="IMU-I2C" gate="G$1" pin="5"/>
-<wire x1="53.34" y1="134.62" x2="53.34" y2="124.46" width="0.1524" layer="91"/>
+<wire x1="53.34" y1="162.56" x2="53.34" y2="124.46" width="0.1524" layer="91"/>
 <junction x="53.34" y="124.46"/>
-<pinref part="SV1" gate="1" pin="4"/>
-<wire x1="43.18" y1="152.4" x2="58.42" y2="152.4" width="0.1524" layer="91"/>
-<wire x1="58.42" y1="152.4" x2="58.42" y2="124.46" width="0.1524" layer="91"/>
-<junction x="58.42" y="124.46"/>
 <wire x1="-55.88" y1="-17.78" x2="-55.88" y2="-22.86" width="0.1524" layer="91"/>
 <junction x="-55.88" y="-22.86"/>
@@
 <pinref part="PRJ1" gate="G$1" pin="19/A5/SCL"/>
 <pinref part="IMU-I2C" gate="G$1" pin="2"/>
-<wire x1="45.72" y1="114.3" x2="45.72" y2="134.62" width="0.1524" layer="91"/>
+<wire x1="45.72" y1="114.3" x2="45.72" y2="162.56" width="0.1524" layer="91"/>
 <label x="45.72" y="127" size="1.778" layer="95" rot="R270"/>
 </segment>
@@
 <pinref part="PRJ1" gate="G$1" pin="18/A4/SDA"/>
 <pinref part="IMU-I2C" gate="G$1" pin="3"/>
-<wire x1="48.26" y1="114.3" x2="48.26" y2="134.62" width="0.1524" layer="91"/>
+<wire x1="48.26" y1="114.3" x2="48.26" y2="162.56" width="0.1524" layer="91"/>
 <label x="48.26" y="124.46" size="1.778" layer="95" rot="R270"/>
 </segment>
@@
 <wire x1="33.02" y1="132.08" x2="50.8" y2="132.08" width="0.1524" layer="91"/>
 <pinref part="IMU-I2C" gate="G$1" pin="4"/>
-<wire x1="50.8" y1="132.08" x2="50.8" y2="134.62" width="0.1524" layer="91"/>
+<wire x1="50.8" y1="132.08" x2="50.8" y2="162.56" width="0.1524" layer="91"/>
 </segment>
 </net>
@@
 <pinref part="IMU-I2C" gate="G$1" pin="1"/>
 <pinref part="PRJ1" gate="G$1" pin="20/A6"/>
-<wire x1="43.18" y1="134.62" x2="43.18" y2="114.3" width="0.1524" layer="91"/>
-</segment>
-</net>
-<net name="N$49" class="0">
-<segment>
-<pinref part="SV1" gate="1" pin="1"/>
-<pinref part="PRJ1" gate="G$1" pin="23/A9"/>
-<wire x1="35.56" y1="152.4" x2="35.56" y2="114.3" width="0.1524" layer="91"/>
-</segment>
-</net>
-<net name="N$50" class="0">
-<segment>
-<pinref part="SV1" gate="1" pin="2"/>
-<pinref part="PRJ1" gate="G$1" pin="22/A8"/>
-<wire x1="38.1" y1="152.4" x2="38.1" y2="114.3" width="0.1524" layer="91"/>
-</segment>
-</net>
-<net name="N$51" class="0">
-<segment>
-<pinref part="SV1" gate="1" pin="3"/>
-<pinref part="PRJ1" gate="G$1" pin="21/A7"/>
-<wire x1="40.64" y1="152.4" x2="40.64" y2="114.3" width="0.1524" layer="91"/>
+<wire x1="43.18" y1="162.56" x2="43.18" y2="114.3" width="0.1524" layer="91"/>
 </segment>
 </net>
@@
 </segment>
 </net>
+<net name="N$57" class="0">
+<segment>
+<pinref part="HE1" gate="-2" pin="S"/>
+<wire x1="-33.02" y1="76.2" x2="25.4" y2="76.2" width="0.1524" layer="91"/>
+<wire x1="25.4" y1="76.2" x2="25.4" y2="58.42" width="0.1524" layer="91"/>
+<wire x1="25.4" y1="58.42" x2="33.02" y2="58.42" width="0.1524" layer="91"/>
+<pinref part="PRJ1" gate="G$1" pin="1/TX"/>
+<wire x1="33.02" y1="58.42" x2="33.02" y2="73.66" width="0.1524" layer="91"/>
+</segment>
+</net>
+<net name="N$58" class="0">
+<segment>
+<pinref part="HE1" gate="-3" pin="S"/>
+<wire x1="-33.02" y1="78.74" x2="5.08" y2="78.74" width="0.1524" layer="91"/>
+<wire x1="5.08" y1="78.74" x2="5.08" y2="139.7" width="0.1524" layer="91"/>
+<wire x1="5.08" y1="139.7" x2="58.42" y2="139.7" width="0.1524" layer="91"/>
+<pinref part="PRJ1" gate="G$1" pin="14/A0"/>
+<wire x1="58.42" y1="139.7" x2="58.42" y2="114.3" width="0.1524" layer="91"/>
+</segment>
+</net>
+<net name="N$49" class="0">
+<segment>
+<pinref part="PRJ1" gate="G$1" pin="23/A9"/>
+<wire x1="35.56" y1="114.3" x2="35.56" y2="127" width="0.1524" layer="91"/>
+<wire x1="35.56" y1="127" x2="-15.24" y2="127" width="0.1524" layer="91"/>
+<pinref part="HE3" gate="-2" pin="S"/>
+<wire x1="-15.24" y1="127" x2="-15.24" y2="111.76" width="0.1524" layer="91"/>
+<wire x1="-15.24" y1="111.76" x2="-33.02" y2="111.76" width="0.1524" layer="91"/>
+</segment>
+</net>
+<net name="N$50" class="0">
+<segment>
+<pinref part="HE3" gate="-3" pin="S"/>
+<wire x1="-33.02" y1="114.3" x2="-17.78" y2="114.3" width="0.1524" layer="91"/>
+<wire x1="-17.78" y1="114.3" x2="-17.78" y2="129.54" width="0.1524" layer="91"/>
+<wire x1="-17.78" y1="129.54" x2="38.1" y2="129.54" width="0.1524" layer="91"/>
+<pinref part="PRJ1" gate="G$1" pin="22/A8"/>
+<wire x1="38.1" y1="129.54" x2="38.1" y2="114.3" width="0.1524" layer="91"/>
+</segment>
+</net>
+<net name="N$51" class="0">
+<segment>
+<pinref part="PRJ1" gate="G$1" pin="21/A7"/>
+<wire x1="40.64" y1="114.3" x2="40.64" y2="134.62" width="0.1524" layer="91"/>
+<wire x1="40.64" y1="134.62" x2="-20.32" y2="134.62" width="0.1524" layer="91"/>
+<wire x1="-20.32" y1="134.62" x2="-20.32" y2="93.98" width="0.1524" layer="91"/>
+<pinref part="HE2" gate="-2" pin="S"/>
+<wire x1="-20.32" y1="93.98" x2="-33.02" y2="93.98" width="0.1524" layer="91"/>
+</segment>
+</net>
+<net name="N$59" class="0">
+<segment>
+<pinref part="HE2" gate="-3" pin="S"/>
+<wire x1="-33.02" y1="96.52" x2="-22.86" y2="96.52" width="0.1524" layer="91"/>
+<wire x1="-22.86" y1="96.52" x2="-22.86" y2="137.16" width="0.1524" layer="91"/>
+<wire x1="-22.86" y1="137.16" x2="60.96" y2="137.16" width="0.1524" layer="91"/>
+<pinref part="PRJ1" gate="G$1" pin="13/SCK"/>
+<wire x1="60.96" y1="137.16" x2="60.96" y2="114.3" width="0.1524" layer="91"/>
+</segment>
+</net>

Commit message: no message
Parts:
- removed CONTROL-I2C, LOG-UART: 1, con-lstb:MA03-1
- added CONTROL: (no value), con-lstb:MA06-1
- added U$2: LEVEL-SHIFTER-4CHLEVEL-SHIFTER-4CH-ADAFRUIT, diy-modules:LEVEL-SHIFTER-4CHLEVEL-SHIFTER-4CH-ADAFRUIT
Connections:
- removed net CTRL-SDA: CONTROL-I2C.1, PRJ1.37/A18
- removed net N$43: CONTROL-I2C.2, PRJ1.38/A19
- removed net N$53: HE1-5.S, HE2-5.S, HE3-5.S
- new net LCTR-VDD: CONTROL.6, U$2.HV4
- new net LCTRL-GND: CONTROL.1, U$2.GND.2
- new net LCTRL-RX: CONTROL.5, U$2.HV3
- new net LCTRL-SCL: CONTROL.4, U$2.HV2
- new net LCTRL-SDA: CONTROL.3, U$2.HV1
- new net LCTRL-VDD: CONTROL.2, U$2.HV
- new net N$60: PRJ1.A22/DAC1, U$1.FB
- new net SCL1: PRJ1.38/A19, U$2.LV1
- new net SDA1: PRJ1.37/A18, U$2.LV2
- net GND: now also PRJ1.AGND, PRJ1.GND2, U$2.GND.1; no longer CONTROL-I2C.3, LOG-UART.3
- net LIPO-GND: now also U$1.D1
- net N$46: now also HE1-5.S, HE2-5.S, HE3-5.S
- net RX5: now also U$2.LV4; no longer LOG-UART.1
- net TX5: now also U$2.LV3; no longer LOG-UART.2
- net VCC: now also U$1.!D2

Commit message: ordered PCB
Parts:
- D1: value 1N5400 -> 1N5908; device diode:1N5400 -> diode:1N5908
- D2: value 1N4148DO35-7 -> 1N5818-B; device diode:1N4148DO35-7 -> diode:1N5818-B
Connections:
- net GND: no longer PRJ1.AGND, PRJ1.GND2
Other:
- moved on the sheet: REL1
Changed lines of the file:
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@@
 <part name="IMU-I2C" library="con-lstb" library_urn="urn:adsk.eagle:library:162" deviceset="MA05-1" device="" package3d_urn="urn:adsk.eagle:package:8332/1" value="1"/>
 <part name="DC-MOTOR" library="con-lstb" library_urn="urn:adsk.eagle:library:162" deviceset="MA06-1" device="" package3d_urn="urn:adsk.eagle:package:8340/1" value="1"/>
-<part name="D1" library="diode" library_urn="urn:adsk.eagle:library:210" deviceset="1N5400" device="" package3d_urn="urn:adsk.eagle:package:43365/1"/>
+<part name="D1" library="diode" library_urn="urn:adsk.eagle:library:210" deviceset="1N5908" device="" package3d_urn="urn:adsk.eagle:package:43355/1"/>
 <part name="C1" library="rcl" library_urn="urn:adsk.eagle:library:334" deviceset="CPOL-EU" device="E7.5-16" package3d_urn="urn:adsk.eagle:package:23382/2" value="470uF"/>
 <part name="C2" library="rcl" library_urn="urn:adsk.eagle:library:334" deviceset="CPOL-EU" device="E7.5-16" package3d_urn="urn:adsk.eagle:package:23382/2" value="470uF"/>
@@
 <part name="IC1" library="v-reg" library_urn="urn:adsk.eagle:library:409" deviceset="78XXL" device="" package3d_urn="urn:adsk.eagle:package:30361/1" value="7805"/>
 <part name="POWER_IN" library="SparkFun-Connectors" library_urn="urn:adsk.eagle:library:513" deviceset="CONN_02" device="3.5MM" package3d_urn="urn:adsk.eagle:package:38050/1" value="12V"/>
-<part name="D2" library="diode" library_urn="urn:adsk.eagle:library:210" deviceset="1N4148" device="DO35-7" package3d_urn="urn:adsk.eagle:package:43339/1"/>
+<part name="D2" library="diode" library_urn="urn:adsk.eagle:library:210" deviceset="1N581*" device="" package3d_urn="urn:adsk.eagle:package:43421/1" technology="8-B"/>
 <part name="Q1" library="transistor-pnp" library_urn="urn:adsk.eagle:library:399" deviceset="BC307" device="" package3d_urn="urn:adsk.eagle:package:29211/2"/>
 <part name="R11" library="resistor" library_urn="urn:adsk.eagle:library:348" deviceset="R-EU_" device="0204/2V" package3d_urn="urn:adsk.eagle:package:23495/1" value="0"/>
@@
 <instance part="IC1" gate="A" x="-109.22" y="45.72"/>
 <instance part="POWER_IN" gate="G$1" x="-142.24" y="55.88"/>
-<instance part="D2" gate="G$1" x="-45.72" y="-12.7" rot="R90"/>
+<instance part="D2" gate="G$1" x="-45.72" y="-17.78" rot="R90"/>
 <instance part="Q1" gate="G$1" x="-58.42" y="7.62"/>
 <instance part="R11" gate="G$1" x="-121.92" y="-30.48" rot="R90"/>
@@
 <wire x1="175.26" y1="48.26" x2="175.26" y2="-22.86" width="0.1524" layer="91"/>
 <junction x="175.26" y="48.26"/>
-<wire x1="53.34" y1="124.46" x2="63.5" y2="124.46" width="0.1524" layer="91"/>
-<wire x1="63.5" y1="124.46" x2="73.66" y2="124.46" width="0.1524" layer="91"/>
-<wire x1="53.34" y1="124.46" x2="30.48" y2="124.46" width="0.1524" layer="91"/>
-<wire x1="30.48" y1="124.46" x2="17.78" y2="124.46" width="0.1524" layer="91"/>
+<wire x1="53.34" y1="124.46" x2="17.78" y2="124.46" width="0.1524" layer="91"/>
 <wire x1="17.78" y1="124.46" x2="15.24" y2="124.46" width="0.1524" layer="91"/>
 <wire x1="15.24" y1="124.46" x2="-12.7" y2="124.46" width="0.1524" layer="91"/>
@@
 <wire x1="-78.74" y1="25.4" x2="-78.74" y2="-22.86" width="0.1524" layer="91"/>
 <junction x="-78.74" y="-22.86"/>
-<wire x1="93.98" y1="124.46" x2="73.66" y2="124.46" width="0.1524" layer="91"/>
+<wire x1="101.6" y1="124.46" x2="53.34" y2="124.46" width="0.1524" layer="91"/>
 <pinref part="IC1" gate="A" pin="GND"/>
 <wire x1="-109.22" y1="38.1" x2="-109.22" y2="-22.86" width="0.1524" layer="91"/>
@@
 <junction x="-55.88" y="-22.86"/>
 <pinref part="D2" gate="G$1" pin="A"/>
-<wire x1="-45.72" y1="-15.24" x2="-45.72" y2="-22.86" width="0.1524" layer="91"/>
+<wire x1="-45.72" y1="-20.32" x2="-45.72" y2="-22.86" width="0.1524" layer="91"/>
 <junction x="-45.72" y="-22.86"/>
 <pinref part="R11" gate="G$1" pin="2"/>
@@
 <wire x1="228.6" y1="124.46" x2="101.6" y2="124.46" width="0.1524" layer="91"/>
 <pinref part="S1" gate="1" pin="1"/>
-<wire x1="101.6" y1="124.46" x2="93.98" y2="124.46" width="0.1524" layer="91"/>
 <wire x1="15.24" y1="127" x2="15.24" y2="124.46" width="0.1524" layer="91"/>
 <junction x="15.24" y="124.46"/>
@@
 <pinref part="U$2" gate="G$1" pin="GND.1"/>
 <wire x1="71.12" y1="167.64" x2="66.04" y2="167.64" width="0.1524" layer="91"/>
-<wire x1="66.04" y1="167.64" x2="66.04" y2="154.94" width="0.1524" layer="91"/>
-<wire x1="66.04" y1="154.94" x2="66.04" y2="152.4" width="0.1524" layer="91"/>
+<wire x1="66.04" y1="167.64" x2="66.04" y2="152.4" width="0.1524" layer="91"/>
 <wire x1="66.04" y1="152.4" x2="101.6" y2="152.4" width="0.1524" layer="91"/>
 <wire x1="101.6" y1="152.4" x2="101.6" y2="124.46" width="0.1524" layer="91"/>
 <junction x="101.6" y="124.46"/>
-<pinref part="PRJ1" gate="G$1" pin="AGND"/>
-<wire x1="30.48" y1="114.3" x2="30.48" y2="124.46" width="0.1524" layer="91"/>
-<junction x="30.48" y="124.46"/>
-<pinref part="PRJ1" gate="G$1" pin="GND2"/>
-<wire x1="63.5" y1="114.3" x2="63.5" y2="124.46" width="0.1524" layer="91"/>
-<junction x="63.5" y="124.46"/>
 </segment>
 </net>
@@
 <pinref part="D2" gate="G$1" pin="C"/>
 <wire x1="-55.88" y1="-7.62" x2="-45.72" y2="-7.62" width="0.1524" layer="91"/>
-<wire x1="-45.72" y1="-7.62" x2="-45.72" y2="-10.16" width="0.1524" layer="91"/>
+<wire x1="-45.72" y1="-7.62" x2="-45.72" y2="-15.24" width="0.1524" layer="91"/>
 <wire x1="-55.88" y1="2.54" x2="-55.88" y2="-7.62" width="0.1524" layer="91"/>
 <pinref part="Q1" gate="G$1" pin="C"/>
