File: schematics/MotorController V2.sch (EAGLE design)
At the start: 40 parts, among them IC1 7805, Q1 BC307

Commit message: AfterWeekend
Parts:
- removed HALL1, HALL2, HALL3: (no value), con-molex-micro-fit-3_0:HEADER_POS6_43045-0612
- added D10, D11, D12, D13, D4, D5, D6, D7, D8, D9: 5.1V, diode:ZENER-DIODEDO41Z10
- added D3: 1N5818-B, diode:1N5818-B
- added R12, R13, R14: 1K, resistor:R-EU_0204/7
- C1: value 2200uF -> 1000uF; device rcl:CPOL-EUE7.5-16 -> rcl:CPOL-EUE5-10.5
- C2: value 2200uF -> 100uF; device rcl:CPOL-EUE7.5-16 -> rcl:CPOL-EUE5-5
- CONTROL, S1, S2: value (none) -> (none)
- R1, R2, R3: value 330 -> 1K
Connections:
- net N$48 renamed IMU-INT
- removed net LCTR-RX: CONTROL.6, U$2.HV4
- removed net LCTRL-GND: CONTROL.1, U$2.GND.2
- removed net LCTRL-SCL: CONTROL.4, U$2.HV2
- removed net LCTRL-SDA: CONTROL.3, U$2.HV1
- removed net LCTRL-TX: CONTROL.5, U$2.HV3
- removed net LCTRL-VDD: CONTROL.2, U$2.HV
- removed net N$49: HALL3.2, PRJ1.23/A9
- removed net N$50: HALL3.3, PRJ1.22/A8
- removed net N$51: HALL2.2, PRJ1.21/A7
- removed net N$54: HALL1.1, PRJ1.17/A3
- removed net N$55: HALL2.1, PRJ1.16/A2
- removed net N$56: HALL3.1, PRJ1.15/A1
- removed net N$57: HALL1.2, PRJ1.1/TX
- removed net N$58: HALL1.3, PRJ1.14/A0
- removed net N$59: HALL2.3, PRJ1.13/SCK
- new net CTR-SCL: CONTROL.4, U$2.LV1
- new net CTR-SDA: CONTROL.3, U$2.LV2
- new net CTRL-GND: CONTROL.1, U$2.GND.1
- new net CTRL-RX: CONTROL.6, U$2.LV4
- new net CTRL-TX: CONTROL.5, U$2.LV3
- new net CTRL-VDD: CONTROL.2, U$2.LV
- new net N$43: DRK1.EN, R12.2
- new net N$46: D4.C, PRJ1.24, R12.1, R13.1, R14.1
- new net N$48: DRK2.EN, R13.2
- net 3.3V: now also U$2.HV; no longer HALL1.5, HALL2.5, HALL3.5
- net GND: now also D10.A, D11.A, D12.A, D13.A, D4.A, D5.A, D6.A, D7.A, D8.A, D9.A, U$2.GND.2; no longer HALL1.4, HALL2.4, HALL3.4, U$2.GND.1
- net IMU-SCL: now also PRJ1.18/A4/SDA; no longer PRJ1.19/A5/SCL
- net IMU-SDA: now also PRJ1.19/A5/SCL; no longer PRJ1.18/A4/SDA
- net N$10: now also R14.2; no longer DRK1.EN, DRK2.EN, PRJ1.24
- net N$21: now also D8.C
- net N$22: now also D9.C
- net N$23: now also D10.C
- net N$27: now also D11.C
- net N$28: now also D12.C
- net N$29: now also D13.C
- net N$32: now also D3.C
- net N$34: now also ENCODER1.1; no longer ENCODER1.2
- net N$36: now also ENCODER2.1; no longer ENCODER2.2
- net N$38: now also ENCODER3.1; no longer ENCODER3.2
- net N$7: now also D7.C
- net N$8: now also D6.C
- net N$9: now also D5.C
- net RX5: now also U$2.HV4; no longer U$2.LV4
- net SCL1: now also U$2.HV1; no longer U$2.LV1
- net SDA1: now also U$2.HV2; no longer U$2.LV2
- net TX5: now also U$2.HV3; no longer U$2.LV3
- net VCC: now also D3.A, ENCODER1.2, ENCODER2.2, ENCODER3.2; no longer ENCODER1.1, ENCODER2.1, ENCODER3.1
Other:
- moved on the sheet: C3, ENCODER1, IMU-I2C, S1
