File: schematics/MotorController V2.sch (EAGLE design)
At the start: 51 parts, among them IC1 7805, Q1 BC307

Commit message: no message
Parts:
- D10, D11, D12, D13, D4, D5, D6, D7, D8, D9: value 5.1V -> 5.6V
Connections:
- removed net N$41: PRJ1.32/A13, U$1.INV
- net LIPO-GND: no longer U$1.D1
- net VCC: no longer U$1.!D2
Other:
- moved on the sheet: D10, D11, D13, D4, D6, D8, R1, R13, R14, R3, R4, R5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

Commit message: accelerated bldc setup
Parts:
- CONTROL: device con-lstb:MA06-1 -> con-lstb:MA08-1
- IC1: device v-reg:78XXL -> v-reg:78XXS
Connections:
- removed net 3.3V: IMU-I2C.4, PRJ1.3V3_LO, U$2.HV
- removed net VCC: C1.+, C3.1, D3.A, DC-MOTOR.4, ENCODER1.2, ENCODER2.2, ENCODER3.2, IC1.OUT, PRJ1.VIN, Q1.E, U$1.VDD(+5V)
- new net CTRL-3.3V: CONTROL.7, IMU-I2C.4, PRJ1.3V3_LO, U$2.HV
- new net CTRL-5.0V: C1.+, C3.1, CONTROL.8, D3.A, DC-MOTOR.4, ENCODER1.2, ENCODER2.2, ENCODER3.2, IC1.OUT, PRJ1.VIN, Q1.E, U$1.VDD(+5V)
Other:
- moved on the sheet: U$1
Changed lines of the file:
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@@
 <part name="MOTOR2" library="con-molex" library_urn="urn:adsk.eagle:library:165" deviceset="5566-4" device=""/>
 <part name="MOTOR3" library="con-molex" library_urn="urn:adsk.eagle:library:165" deviceset="5566-4" device=""/>
-<part name="IC1" library="v-reg" library_urn="urn:adsk.eagle:library:409" deviceset="78XXL" device="" package3d_urn="urn:adsk.eagle:package:30361/1" value="7805"/>
+<part name="IC1" library="v-reg" library_urn="urn:adsk.eagle:library:409" deviceset="78XXS" device="" package3d_urn="urn:adsk.eagle:package:30342/1" value="7805"/>
 <part name="POWER_IN" library="SparkFun-Connectors" library_urn="urn:adsk.eagle:library:513" deviceset="CONN_02" device="3.5MM" package3d_urn="urn:adsk.eagle:package:38050/1" value="12V"/>
 <part name="D2" library="diode" library_urn="urn:adsk.eagle:library:210" deviceset="1N581*" device="" package3d_urn="urn:adsk.eagle:package:43421/1" technology="8-B"/>
@@
 <part name="S2" library="switch-omron" library_urn="urn:adsk.eagle:library:377" deviceset="10-XX" device="" package3d_urn="urn:adsk.eagle:package:27496/1" value=" "/>
 <part name="U$2" library="diy-modules" deviceset="LEVEL-SHIFTER-4CH" device="LEVEL-SHIFTER-4CH-ADAFRUIT"/>
-<part name="CONTROL" library="con-lstb" library_urn="urn:adsk.eagle:library:162" deviceset="MA06-1" device="" package3d_urn="urn:adsk.eagle:package:8340/1" value=" "/>
+<part name="CONTROL" library="con-lstb" library_urn="urn:adsk.eagle:library:162" deviceset="MA08-1" device="" package3d_urn="urn:adsk.eagle:package:8343/1" value=" "/>
 <part name="D3" library="diode" library_urn="urn:adsk.eagle:library:210" deviceset="1N581*" device="" package3d_urn="urn:adsk.eagle:package:43421/1" technology="8-B"/>
 <part name="R12" library="resistor" library_urn="urn:adsk.eagle:library:348" deviceset="R-EU_" device="0204/7" package3d_urn="urn:adsk.eagle:package:23498/1" value="1K"/>
@@
 <instance part="MOTOR3" gate="-3" x="167.64" y="-12.7" rot="R270"/>
 <instance part="MOTOR3" gate="-4" x="165.1" y="-12.7" rot="R270"/>
-<instance part="IC1" gate="A" x="-109.22" y="45.72"/>
+<instance part="IC1" gate="1" x="-109.22" y="45.72"/>
 <instance part="POWER_IN" gate="G$1" x="-142.24" y="55.88"/>
 <instance part="D2" gate="G$1" x="-45.72" y="-17.78" rot="R90"/>
@@
 <instance part="S2" gate="1" x="119.38" y="99.06" rot="R270"/>
 <instance part="U$2" gate="G$1" x="86.36" y="170.18" rot="MR0"/>
-<instance part="CONTROL" gate="1" x="121.92" y="170.18"/>
+<instance part="CONTROL" gate="1" x="127" y="170.18"/>
 <instance part="D3" gate="G$1" x="-109.22" y="50.8" rot="R180"/>
 <instance part="R12" gate="G$1" x="15.24" y="5.08"/>
@@
 </busses>
 <nets>
-<net name="VCC" class="0">
+<net name="CTRL-5.0V" class="0">
 <segment>
 <pinref part="P+1" gate="VCC" pin="VCC"/>
@@
 <wire x1="177.8" y1="76.2" x2="177.8" y2="91.44" width="0.1524" layer="91"/>
 <wire x1="177.8" y1="91.44" x2="177.8" y2="93.98" width="0.1524" layer="91"/>
-<wire x1="27.94" y1="149.86" x2="177.8" y2="149.86" width="0.1524" layer="91"/>
+<wire x1="27.94" y1="149.86" x2="154.94" y2="149.86" width="0.1524" layer="91"/>
+<wire x1="154.94" y1="149.86" x2="177.8" y2="149.86" width="0.1524" layer="91"/>
 <wire x1="177.8" y1="149.86" x2="177.8" y2="93.98" width="0.1524" layer="91"/>
 <wire x1="-55.88" y1="45.72" x2="-71.12" y2="45.72" width="0.1524" layer="91"/>
@@
 <wire x1="246.38" y1="132.08" x2="213.36" y2="132.08" width="0.1524" layer="91"/>
 <junction x="213.36" y="132.08"/>
-<pinref part="IC1" gate="A" pin="OUT"/>
+<pinref part="IC1" gate="1" pin="OUT"/>
 <junction x="-83.82" y="45.72"/>
 <wire x1="-101.6" y1="45.72" x2="-91.44" y2="45.72" width="0.1524" layer="91"/>
@@
 <wire x1="-106.68" y1="50.8" x2="-91.44" y2="50.8" width="0.1524" layer="91"/>
 <wire x1="-91.44" y1="50.8" x2="-91.44" y2="45.72" width="0.1524" layer="91"/>
+<pinref part="CONTROL" gate="1" pin="8"/>
+<wire x1="134.62" y1="180.34" x2="154.94" y2="180.34" width="0.1524" layer="91"/>
+<wire x1="154.94" y1="180.34" x2="154.94" y2="149.86" width="0.1524" layer="91"/>
+<junction x="154.94" y="149.86"/>
+<label x="134.62" y="180.34" size="1.778" layer="95"/>
 </segment>
 </net>
@@
 <wire x1="-91.44" y1="25.4" x2="-91.44" y2="-22.86" width="0.1524" layer="91"/>
 <junction x="-91.44" y="-22.86"/>
-<pinref part="IC1" gate="A" pin="GND"/>
+<pinref part="IC1" gate="1" pin="GND"/>
 <wire x1="-109.22" y1="38.1" x2="-109.22" y2="-22.86" width="0.1524" layer="91"/>
 <junction x="-109.22" y="-22.86"/>
@@
 <pinref part="C2" gate="G$1" pin="+"/>
 <wire x1="-121.92" y1="35.56" x2="-121.92" y2="45.72" width="0.1524" layer="91"/>
-<pinref part="IC1" gate="A" pin="IN"/>
+<pinref part="IC1" gate="1" pin="IN"/>
 <wire x1="-116.84" y1="45.72" x2="-121.92" y2="45.72" width="0.1524" layer="91"/>
 <wire x1="-121.92" y1="58.42" x2="-121.92" y2="50.8" width="0.1524" layer="91"/>
@@
 <segment>
 <pinref part="CONTROL" gate="1" pin="6"/>
-<wire x1="129.54" y1="175.26" x2="129.54" y2="180.34" width="0.1524" layer="91"/>
-<wire x1="129.54" y1="180.34" x2="106.68" y2="180.34" width="0.1524" layer="91"/>
+<wire x1="124.46" y1="180.34" x2="106.68" y2="180.34" width="0.1524" layer="91"/>
 <wire x1="106.68" y1="180.34" x2="106.68" y2="162.56" width="0.1524" layer="91"/>
 <pinref part="U$2" gate="G$1" pin="LV4"/>
 <wire x1="106.68" y1="162.56" x2="101.6" y2="162.56" width="0.1524" layer="91"/>
-<label x="129.54" y="175.26" size="1.778" layer="95"/>
+<label x="134.62" y="175.26" size="1.778" layer="95"/>
+<wire x1="124.46" y1="180.34" x2="124.46" y2="175.26" width="0.1524" layer="91"/>
+<wire x1="124.46" y1="175.26" x2="134.62" y2="175.26" width="0.1524" layer="91"/>
 </segment>
 </net>
@@
 <wire x1="121.92" y1="177.8" x2="121.92" y2="172.72" width="0.1524" layer="91"/>
 <pinref part="CONTROL" gate="1" pin="5"/>
-<wire x1="121.92" y1="172.72" x2="129.54" y2="172.72" width="0.1524" layer="91"/>
+<wire x1="121.92" y1="172.72" x2="134.62" y2="172.72" width="0.1524" layer="91"/>
 <wire x1="121.92" y1="177.8" x2="109.22" y2="177.8" width="0.1524" layer="91"/>
 <wire x1="109.22" y1="177.8" x2="109.22" y2="165.1" width="0.1524" layer="91"/>
 <pinref part="U$2" gate="G$1" pin="LV3"/>
 <wire x1="109.22" y1="165.1" x2="101.6" y2="165.1" width="0.1524" layer="91"/>
-<label x="129.54" y="172.72" size="1.778" layer="95"/>
+<label x="134.62" y="172.72" size="1.778" layer="95"/>
 </segment>
 </net>
@@
 </segment>
 </net>
-<net name="3.3V" class="0">
+<net name="CTRL-3.3V" class="0">
 <segment>
 <pinref part="PRJ1" gate="G$1" pin="3V3_LO"/>
@@
 <wire x1="33.02" y1="132.08" x2="50.8" y2="132.08" width="0.1524" layer="91"/>
 <pinref part="IMU-I2C" gate="G$1" pin="4"/>
-<wire x1="50.8" y1="132.08" x2="50.8" y2="157.48" width="0.1524" layer="91"/>
+<wire x1="50.8" y1="132.08" x2="50.8" y2="152.4" width="0.1524" layer="91"/>
+<wire x1="50.8" y1="152.4" x2="50.8" y2="157.48" width="0.1524" layer="91"/>
 <wire x1="50.8" y1="157.48" x2="50.8" y2="170.18" width="0.1524" layer="91"/>
 <label x="33.02" y="132.08" size="1.778" layer="95"/>
@@
 <pinref part="U$2" gate="G$1" pin="HV"/>
 <wire x1="58.42" y1="170.18" x2="71.12" y2="170.18" width="0.1524" layer="91"/>
+<pinref part="CONTROL" gate="1" pin="7"/>
+<wire x1="134.62" y1="177.8" x2="152.4" y2="177.8" width="0.1524" layer="91"/>
+<wire x1="152.4" y1="177.8" x2="152.4" y2="152.4" width="0.1524" layer="91"/>
+<wire x1="152.4" y1="152.4" x2="50.8" y2="152.4" width="0.1524" layer="91"/>
+<junction x="50.8" y="152.4"/>
+<label x="134.62" y="177.8" size="1.778" layer="95"/>
 </segment>
 </net>
@@
 <segment>
 <pinref part="CONTROL" gate="1" pin="2"/>
-<wire x1="129.54" y1="165.1" x2="119.38" y2="165.1" width="0.1524" layer="91"/>
-<label x="129.54" y="165.1" size="1.778" layer="95"/>
+<wire x1="134.62" y1="165.1" x2="119.38" y2="165.1" width="0.1524" layer="91"/>
+<label x="134.62" y="165.1" size="1.778" layer="95"/>
 <pinref part="U$2" gate="G$1" pin="LV"/>
 <wire x1="101.6" y1="170.18" x2="114.3" y2="170.18" width="0.1524" layer="91"/>
@@
 <segment>
 <pinref part="CONTROL" gate="1" pin="1"/>
-<wire x1="129.54" y1="162.56" x2="116.84" y2="162.56" width="0.1524" layer="91"/>
-<label x="129.54" y="162.56" size="1.778" layer="95"/>
+<wire x1="134.62" y1="162.56" x2="116.84" y2="162.56" width="0.1524" layer="91"/>
+<label x="134.62" y="162.56" size="1.778" layer="95"/>
 <pinref part="U$2" gate="G$1" pin="GND.1"/>
 <wire x1="101.6" y1="167.64" x2="111.76" y2="167.64" width="0.1524" layer="91"/>
@@
 <segment>
 <pinref part="CONTROL" gate="1" pin="4"/>
-<label x="129.54" y="170.18" size="1.778" layer="95"/>
+<label x="134.62" y="170.18" size="1.778" layer="95"/>
 <pinref part="U$2" gate="G$1" pin="LV1"/>
 <wire x1="101.6" y1="175.26" x2="119.38" y2="175.26" width="0.1524" layer="91"/>
 <wire x1="119.38" y1="175.26" x2="119.38" y2="170.18" width="0.1524" layer="91"/>
-<wire x1="119.38" y1="170.18" x2="129.54" y2="170.18" width="0.1524" layer="91"/>
+<wire x1="119.38" y1="170.18" x2="134.62" y2="170.18" width="0.1524" layer="91"/>
 </segment>
 </net>
 <net name="CTR-SDA" class="0">
 <segment>
-<wire x1="121.92" y1="167.64" x2="116.84" y2="167.64" width="0.1524" layer="91"/>
+<wire x1="129.54" y1="167.64" x2="116.84" y2="167.64" width="0.1524" layer="91"/>
 <wire x1="116.84" y1="167.64" x2="116.84" y2="172.72" width="0.1524" layer="91"/>
 <pinref part="U$2" gate="G$1" pin="LV2"/>
 <wire x1="116.84" y1="172.72" x2="101.6" y2="172.72" width="0.1524" layer="91"/>
 <pinref part="CONTROL" gate="1" pin="3"/>
-<wire x1="121.92" y1="167.64" x2="129.54" y2="167.64" width="0.1524" layer="91"/>
-<label x="129.54" y="167.64" size="1.778" layer="95"/>
-</segment>
-</net>
+<wire x1="129.54" y1="167.64" x2="134.62" y2="167.64" width="0.1524" layer="91"/>
+<label x="134.62" y="167.64" size="1.778" layer="95"/>
+</segment>
+</net>

Commit message: no message
Parts:
- added U$3: NODEMCU, nodemcu:NODEMCU
Changed lines of the file:
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@@
 <part name="D12" library="diode" library_urn="urn:adsk.eagle:library:210" deviceset="ZENER-DIODE" device="DO41Z10" package3d_urn="urn:adsk.eagle:package:43341/1" value="5.6V"/>
 <part name="D13" library="diode" library_urn="urn:adsk.eagle:library:210" deviceset="ZENER-DIODE" device="DO41Z10" package3d_urn="urn:adsk.eagle:package:43341/1" value="5.6V"/>
+<part name="U$3" library="nodemcu" deviceset="NODEMCU" device=""/>
 </parts>
 <sheets>
@@
 <instance part="D12" gate="G$1" x="127" y="-10.16" rot="R90"/>
 <instance part="D13" gate="G$1" x="132.08" y="-15.24" rot="R90"/>
+<instance part="U$3" gate="G$1" x="147.32" y="226.06" rot="R180"/>
 </instances>
 <busses>

Commit message: i2c between webserver and bot controller
Parts:
- removed U$2: LEVEL-SHIFTER-4CHLEVEL-SHIFTER-4CH-ADAFRUIT, diy-modules:LEVEL-SHIFTER-4CHLEVEL-SHIFTER-4CH-ADAFRUIT
Connections:
- removed net CTR-SCL: CONTROL.4, U$2.LV1
- removed net CTR-SDA: CONTROL.3, U$2.LV2
- removed net CTRL-GND: CONTROL.1, U$2.GND.1
- removed net CTRL-RX: CONTROL.6, U$2.LV4
- removed net CTRL-TX: CONTROL.5, U$2.LV3
- removed net CTRL-VDD: CONTROL.2, U$2.LV
- net CTRL-3.3V: no longer U$2.HV
- net CTRL-5.0V: now also U$3.VIN
- net GND: now also U$3.GND@2, U$3.GND@3, U$3.GND@4; no longer U$2.GND.2
- net RX5: no longer U$2.HV4
- net SCL1: now also U$3.D2; no longer U$2.HV1
- net SDA1: now also U$3.D1; no longer U$2.HV2
- net TX5: no longer U$2.HV3

Commit message: updated
Parts:
- added LED1: (no value), led:LED3MM
- added R15: 4,7K, resistor:R-EU_0204/7
Connections:
- new net N$41: LED1.A, R15.2
- net CTRL-3.3V: now also CONTROL.2; no longer CONTROL.7
- net CTRL-5.0V: now also CONTROL.3; no longer CONTROL.8
- net GND: now also CONTROL.1, R15.1
- net LIPO-VDD: now also LED1.C
- net RX5: now also CONTROL.5
- net TX5: now also CONTROL.4, U$3.RX
Changed lines of the file:
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@@
 <part name="D13" library="diode" library_urn="urn:adsk.eagle:library:210" deviceset="ZENER-DIODE" device="DO41Z10" package3d_urn="urn:adsk.eagle:package:43341/1" value="5.6V"/>
 <part name="U$3" library="nodemcu" deviceset="NODEMCU" device=""/>
+<part name="LED1" library="led" library_urn="urn:adsk.eagle:library:259" deviceset="LED" device="3MM" package3d_urn="urn:adsk.eagle:package:15797/1"/>
+<part name="R15" library="resistor" library_urn="urn:adsk.eagle:library:348" deviceset="R-EU_" device="0204/7" package3d_urn="urn:adsk.eagle:package:23498/1" value="4,7K"/>
 </parts>
 <sheets>
@@
 <attribute name="VALUE" x="135.509" y="-17.018" size="1.778" layer="96" rot="R90"/>
 </instance>
-<instance part="U$3" gate="G$1" x="88.9" y="205.74" rot="R180"/>
+<instance part="U$3" gate="G$1" x="93.98" y="205.74" rot="R180"/>
+<instance part="LED1" gate="G$1" x="-27.94" y="10.16" rot="R180">
+<attribute name="NAME" x="-31.496" y="14.732" size="1.778" layer="95" rot="R270"/>
+<attribute name="VALUE" x="-33.655" y="14.732" size="1.778" layer="96" rot="R270"/>
+</instance>
+<instance part="R15" gate="G$1" x="-27.94" y="-7.62" rot="R90">
+<attribute name="NAME" x="-29.4386" y="-11.43" size="1.778" layer="95" rot="R90"/>
+<attribute name="VALUE" x="-24.638" y="-11.43" size="1.778" layer="96" rot="R90"/>
+</instance>
 </instances>
 <busses>
@@
 <wire x1="-106.68" y1="50.8" x2="-91.44" y2="50.8" width="0.1524" layer="91"/>
 <wire x1="-91.44" y1="50.8" x2="-91.44" y2="45.72" width="0.1524" layer="91"/>
-<pinref part="CONTROL" gate="1" pin="8"/>
-<wire x1="134.62" y1="180.34" x2="154.94" y2="180.34" width="0.1524" layer="91"/>
-<wire x1="154.94" y1="180.34" x2="154.94" y2="149.86" width="0.1524" layer="91"/>
 <junction x="154.94" y="149.86"/>
-<label x="134.62" y="180.34" size="1.778" layer="95"/>
+<label x="134.62" y="167.64" size="1.778" layer="95"/>
 <pinref part="U$3" gate="G$1" pin="VIN"/>
-<wire x1="109.22" y1="223.52" x2="121.92" y2="223.52" width="0.1524" layer="91"/>
+<wire x1="154.94" y1="167.64" x2="154.94" y2="149.86" width="0.1524" layer="91"/>
+<wire x1="114.3" y1="223.52" x2="121.92" y2="223.52" width="0.1524" layer="91"/>
 <wire x1="121.92" y1="223.52" x2="121.92" y2="149.86" width="0.1524" layer="91"/>
 <junction x="121.92" y="149.86"/>
+<pinref part="CONTROL" gate="1" pin="3"/>
+<wire x1="134.62" y1="167.64" x2="154.94" y2="167.64" width="0.1524" layer="91"/>
 </segment>
 </net>
@@
 <wire x1="-91.44" y1="-22.86" x2="-55.88" y2="-22.86" width="0.1524" layer="91"/>
 <wire x1="-55.88" y1="-22.86" x2="-45.72" y2="-22.86" width="0.1524" layer="91"/>
-<wire x1="-45.72" y1="-22.86" x2="-12.7" y2="-22.86" width="0.1524" layer="91"/>
+<wire x1="-45.72" y1="-22.86" x2="-27.94" y2="-22.86" width="0.1524" layer="91"/>
+<wire x1="-27.94" y1="-22.86" x2="-12.7" y2="-22.86" width="0.1524" layer="91"/>
 <wire x1="-12.7" y1="-22.86" x2="-10.16" y2="-22.86" width="0.1524" layer="91"/>
 <pinref part="PRJ1" gate="G$1" pin="GND"/>
@@
 <label x="236.22" y="134.62" size="1.778" layer="95"/>
 <wire x1="228.6" y1="134.62" x2="228.6" y2="124.46" width="0.1524" layer="91"/>
-<wire x1="228.6" y1="124.46" x2="119.38" y2="124.46" width="0.1524" layer="91"/>
+<wire x1="228.6" y1="124.46" x2="137.16" y2="124.46" width="0.1524" layer="91"/>
 <pinref part="S1" gate="1" pin="1"/>
+<wire x1="137.16" y1="124.46" x2="119.38" y2="124.46" width="0.1524" layer="91"/>
 <wire x1="119.38" y1="124.46" x2="60.96" y2="124.46" width="0.1524" layer="91"/>
 <wire x1="60.96" y1="124.46" x2="53.34" y2="124.46" width="0.1524" layer="91"/>
@@
 <wire x1="175.26" y1="38.1" x2="190.5" y2="38.1" width="0.1524" layer="91"/>
 <pinref part="U$3" gate="G$1" pin="GND@4"/>
-<wire x1="68.58" y1="203.2" x2="60.96" y2="203.2" width="0.1524" layer="91"/>
+<wire x1="73.66" y1="203.2" x2="60.96" y2="203.2" width="0.1524" layer="91"/>
 <wire x1="60.96" y1="203.2" x2="60.96" y2="124.46" width="0.1524" layer="91"/>
 <junction x="60.96" y="124.46"/>
 <pinref part="U$3" gate="G$1" pin="GND@2"/>
-<wire x1="109.22" y1="220.98" x2="119.38" y2="220.98" width="0.1524" layer="91"/>
+<wire x1="114.3" y1="220.98" x2="119.38" y2="220.98" width="0.1524" layer="91"/>
 <wire x1="119.38" y1="220.98" x2="119.38" y2="124.46" width="0.1524" layer="91"/>
 <junction x="119.38" y="124.46"/>
 <pinref part="U$3" gate="G$1" pin="GND@3"/>
-<wire x1="68.58" y1="220.98" x2="60.96" y2="220.98" width="0.1524" layer="91"/>
+<wire x1="73.66" y1="220.98" x2="60.96" y2="220.98" width="0.1524" layer="91"/>
 <wire x1="60.96" y1="220.98" x2="60.96" y2="203.2" width="0.1524" layer="91"/>
 <junction x="60.96" y="203.2"/>
+<pinref part="CONTROL" gate="1" pin="1"/>
+<wire x1="134.62" y1="162.56" x2="137.16" y2="162.56" width="0.1524" layer="91"/>
+<wire x1="137.16" y1="162.56" x2="137.16" y2="124.46" width="0.1524" layer="91"/>
+<junction x="137.16" y="124.46"/>
+<label x="134.62" y="162.56" size="1.778" layer="95"/>
+<pinref part="R15" gate="G$1" pin="1"/>
+<wire x1="-27.94" y1="-12.7" x2="-27.94" y2="-22.86" width="0.1524" layer="91"/>
+<junction x="-27.94" y="-22.86"/>
 </segment>
 </net>
@@
 <net name="LIPO-VDD" class="1">
 <segment>
-<wire x1="-35.56" y1="25.4" x2="55.88" y2="25.4" width="0.1524" layer="91"/>
+<wire x1="-35.56" y1="25.4" x2="-27.94" y2="25.4" width="0.1524" layer="91"/>
 <pinref part="DRK1" gate="G$1" pin="LIPO+"/>
+<wire x1="-27.94" y1="25.4" x2="55.88" y2="25.4" width="0.1524" layer="91"/>
 <wire x1="55.88" y1="25.4" x2="55.88" y2="15.24" width="0.1524" layer="91"/>
 <wire x1="55.88" y1="25.4" x2="116.84" y2="25.4" width="0.1524" layer="91"/>
@@
 <pinref part="U$1" gate="G$1" pin="VIN(5-28V)"/>
 <pinref part="REL1" gate="G$1" pin="P"/>
+<pinref part="LED1" gate="G$1" pin="C"/>
+<wire x1="-27.94" y1="15.24" x2="-27.94" y2="25.4" width="0.1524" layer="91"/>
+<junction x="-27.94" y="25.4"/>
 </segment>
 </net>
@@
 <wire x1="73.66" y1="154.94" x2="73.66" y2="114.3" width="0.1524" layer="91"/>
 <label x="73.66" y="114.3" size="1.778" layer="95" rot="R90"/>
-<wire x1="73.66" y1="154.94" x2="63.5" y2="154.94" width="0.1524" layer="91"/>
-<wire x1="63.5" y1="154.94" x2="63.5" y2="193.04" width="0.1524" layer="91"/>
+<wire x1="73.66" y1="154.94" x2="68.58" y2="154.94" width="0.1524" layer="91"/>
+<wire x1="68.58" y1="154.94" x2="68.58" y2="193.04" width="0.1524" layer="91"/>
 <pinref part="U$3" gate="G$1" pin="D2"/>
-<wire x1="63.5" y1="193.04" x2="68.58" y2="193.04" width="0.1524" layer="91"/>
+<wire x1="68.58" y1="193.04" x2="73.66" y2="193.04" width="0.1524" layer="91"/>
 </segment>
 </net>
@@
 <label x="76.2" y="114.3" size="1.778" layer="95" rot="R90"/>
 <pinref part="U$3" gate="G$1" pin="D1"/>
-<wire x1="68.58" y1="190.5" x2="66.04" y2="190.5" width="0.1524" layer="91"/>
-<wire x1="66.04" y1="190.5" x2="66.04" y2="157.48" width="0.1524" layer="91"/>
-<wire x1="66.04" y1="157.48" x2="76.2" y2="157.48" width="0.1524" layer="91"/>
+<wire x1="73.66" y1="190.5" x2="71.12" y2="190.5" width="0.1524" layer="91"/>
+<wire x1="71.12" y1="190.5" x2="71.12" y2="157.48" width="0.1524" layer="91"/>
+<wire x1="71.12" y1="157.48" x2="76.2" y2="157.48" width="0.1524" layer="91"/>
 </segment>
 </net>
@@
 <wire x1="50.8" y1="152.4" x2="50.8" y2="170.18" width="0.1524" layer="91"/>
 <label x="33.02" y="132.08" size="1.778" layer="95"/>
-<pinref part="CONTROL" gate="1" pin="7"/>
-<wire x1="134.62" y1="177.8" x2="152.4" y2="177.8" width="0.1524" layer="91"/>
-<wire x1="152.4" y1="177.8" x2="152.4" y2="152.4" width="0.1524" layer="91"/>
+<wire x1="152.4" y1="165.1" x2="152.4" y2="152.4" width="0.1524" layer="91"/>
 <wire x1="152.4" y1="152.4" x2="50.8" y2="152.4" width="0.1524" layer="91"/>
 <junction x="50.8" y="152.4"/>
-<label x="134.62" y="177.8" size="1.778" layer="95"/>
+<label x="134.62" y="165.1" size="1.778" layer="95"/>
+<pinref part="CONTROL" gate="1" pin="2"/>
+<wire x1="134.62" y1="165.1" x2="152.4" y2="165.1" width="0.1524" layer="91"/>
 </segment>
 </net>
@@
 <net name="RX5" class="0">
 <segment>
-<wire x1="83.82" y1="114.3" x2="83.82" y2="162.56" width="0.1524" layer="91"/>
+<wire x1="83.82" y1="114.3" x2="83.82" y2="154.94" width="0.1524" layer="91"/>
 <pinref part="PRJ1" gate="G$1" pin="34/A15"/>
 <label x="83.82" y="119.38" size="1.778" layer="95" rot="R270"/>
+<pinref part="CONTROL" gate="1" pin="5"/>
+<wire x1="134.62" y1="172.72" x2="144.78" y2="172.72" width="0.1524" layer="91"/>
+<wire x1="144.78" y1="172.72" x2="144.78" y2="154.94" width="0.1524" layer="91"/>
+<wire x1="144.78" y1="154.94" x2="83.82" y2="154.94" width="0.1524" layer="91"/>
+<label x="134.62" y="172.72" size="1.778" layer="95"/>
 </segment>
 </net>
@@
 <segment>
 <pinref part="PRJ1" gate="G$1" pin="33/A14"/>
-<wire x1="86.36" y1="114.3" x2="86.36" y2="165.1" width="0.1524" layer="91"/>
+<wire x1="86.36" y1="114.3" x2="86.36" y2="157.48" width="0.1524" layer="91"/>
 <label x="86.36" y="119.38" size="1.778" layer="95" rot="R270"/>
+<wire x1="86.36" y1="157.48" x2="86.36" y2="180.34" width="0.1524" layer="91"/>
+<wire x1="86.36" y1="180.34" x2="63.5" y2="180.34" width="0.1524" layer="91"/>
+<pinref part="U$3" gate="G$1" pin="RX"/>
+<wire x1="73.66" y1="215.9" x2="63.5" y2="215.9" width="0.1524" layer="91"/>
+<wire x1="63.5" y1="180.34" x2="63.5" y2="215.9" width="0.1524" layer="91"/>
+<pinref part="CONTROL" gate="1" pin="4"/>
+<wire x1="134.62" y1="170.18" x2="142.24" y2="170.18" width="0.1524" layer="91"/>
+<wire x1="142.24" y1="170.18" x2="142.24" y2="157.48" width="0.1524" layer="91"/>
+<wire x1="142.24" y1="157.48" x2="86.36" y2="157.48" width="0.1524" layer="91"/>
+<junction x="86.36" y="157.48"/>
+<label x="134.62" y="170.18" size="1.778" layer="95"/>
 </segment>
 </net>
@@
 </segment>
 </net>
+<net name="N$41" class="0">
+<segment>
+<pinref part="R15" gate="G$1" pin="2"/>
+<pinref part="LED1" gate="G$1" pin="A"/>
+<wire x1="-27.94" y1="-2.54" x2="-27.94" y2="7.62" width="0.1524" layer="91"/>
+</segment>
+</net>

Commit message: no message
Parts:
- C1: device rcl:CPOL-EUE5-10.5 -> rcl:CPOL-EUE2.5-6
- LED1: value (none) -> red
Connections:
- net CTRL-3.3V renamed 3.3V
- new net N$49: CONTROL.8, U$3.D0
- new net N$50: CONTROL.7, U$3.RST
- new net N$51: CONTROL.6, PRJ1.14/A0
- net GND: now also U$3.GND, U$3.GND@1
- net SCL1: now also U$3.D1; no longer U$3.D2
- net SDA1: now also U$3.D2; no longer U$3.D1
Other:
- moved on the sheet: DRK3, MOTOR3-1, MOTOR3-2, MOTOR3-3, MOTOR3-4
