File: schematics/MotorController V2.sch (EAGLE design)
At the start: 53 parts, among them IC1 7805, Q1 BC307

Commit message: no message
Connections:
- net IMU-SCL: now also IMU-I2C.3, PRJ1.19/A5/SCL; no longer IMU-I2C.2, PRJ1.18/A4/SDA
- net IMU-SDA: now also IMU-I2C.2, PRJ1.18/A4/SDA; no longer IMU-I2C.3, PRJ1.19/A5/SCL
Changed lines of the file:
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@@
 </segment>
 </net>
-<net name="IMU-SDA" class="0">
+<net name="IMU-SCL" class="0">
 <segment>
 <pinref part="IMU-I2C" gate="G$1" pin="3"/>
@@
 </segment>
 </net>
-<net name="IMU-SCL" class="0">
+<net name="IMU-SDA" class="0">
 <segment>
 <pinref part="IMU-I2C" gate="G$1" pin="2"/>
