File: schematics/MotorController V3.brd (EAGLE design)
At the start: 120.6 x 100 mm, 54 parts, among them IC1 7805, Q1 BC307

Commit message: no message
Parts:
- removed ENCODER1, ENCODER2, ENCODER3: 1, con-lstb:MA04-1
- added ENC0, ENC1, ENC2: (no value), con-lstb:MA06-1
- moved REL1 27.1 mm to (-3.17, 21.6)
- moved D2 14.9 mm to (8.26, 24.8), turned to 90 degrees
- moved Q1 7.96 mm to (-18.4, 22.2)
- moved MOTOR1 5.99 mm to (3.17, -2.54)
- moved U$1 5.46 mm to (25.4, -0.64)
- moved C3 5.43 mm to (5.08, 32.4), turned to 0 degrees
- moved D1 5.08 mm to (-2.54, 35.6)
- moved R10 4.49 mm to (-15.2, 27.3)
- moved C1 3.70 mm to (5.08, 40.0)
- moved MOTOR2 3.59 mm to (-15.2, -3.17)
- moved D14 3.17 mm to (-4.45, 48.3)
- moved MOTOR3 2.62 mm to (-32.4, -3.17)
- moved D4 2.54 mm to (-65.4, 73.0)
- moved R12 2.54 mm to (-52.7, 73.0)
- moved R3 2.54 mm to (-52.7, 70.5)
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Connections:
- removed net +5V: C1.+, C3.1, CONTROL.3, D3.A, DC-MOTOR.4, ENCODER1.2, ENCODER2.2, ENCODER3.2, IC1.OUT, IMU-I2C.4, PRJ1.VIN, Q1.1, U$1.VDD(5V), U$2.30
- removed net ENC1_A: ENCODER1.3, PRJ1.11/MOSI
- removed net ENC1_B: ENCODER1.1, PRJ1.12/MISO
- removed net ENC2_A: ENCODER2.3, PRJ1.25
- removed net ENC2_B: ENCODER2.1, PRJ1.26
- removed net ENC3_A: ENCODER3.3, PRJ1.27
- removed net ENC3_B: ENCODER3.1, PRJ1.28
- new net +3.6V: C1.+, C3.1, CONTROL.3, D3.A, DC-MOTOR.4, IC1.OUT, IMU-I2C.4, PRJ1.VIN, Q1.1, U$1.VDD(5V), U$2.30
- new net CS0: ENC0.2, PRJ1.26
- new net CS1: ENC1.2, PRJ1.25
- new net CS2: ENC2.2, PRJ1.28
- new net MISO: ENC0.5, ENC1.5, ENC2.5, PRJ1.12/MISO
- new net MOSI: ENC0.4, ENC1.4, ENC2.4, PRJ1.11/MOSI
- new net SCK: ENC0.3, ENC1.3, ENC2.3, PRJ1.27
- net 3.3V: now also ENC0.1, ENC1.1, ENC2.1
- net GND: now also ENC0.6, ENC1.6, ENC2.6; no longer ENCODER1.4, ENCODER2.4, ENCODER3.4
Routing:
- net GND: track 404.5 -> 0.00 mm, vias 3 -> 0
- net LIPO-GND: track 338.9 -> 0.00 mm, vias 3 -> 0
- net N$2: track 256.2 -> 0.00 mm, vias 1 -> 0
- net LIPO-VDD: track 224.2 -> 0.00 mm, vias 5 -> 0
- net +5V: track 213.6 -> 0.00 mm, vias 1 -> 0
- net ENC1_A: track 179.7 -> 0.00 mm, vias 1 -> 0
- net SDA1: track 142.7 -> 0.00 mm
- net N$46: track 134.0 -> 0.00 mm
- net N$1: track 130.3 -> 0.00 mm, vias 1 -> 0
- net N$3: track 130.1 -> 0.00 mm, vias 1 -> 0
- net RED-M1: track 129.2 -> 0.00 mm
- net SCL1: track 127.1 -> 0.00 mm
- net N$42: track 120.1 -> 0.00 mm, vias 5 -> 0
- net TX5: track 114.2 -> 0.00 mm, vias 2 -> 0
- net BLCK-M2: track 98.9 -> 0.00 mm, vias 2 -> 0
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
Commit message: forgotten files
Parts:
- moved ENC0 2.84 mm to (1.91, 10.2), turned to 0 degrees
- moved ENC1 2.62 mm to (-15.9, 10.2), turned to 0 degrees
- moved ENC2 2.62 mm to (-33.7, 10.2), turned to 0 degrees
- moved MOTOR3 1.42 mm to (-33.0, -1.91)
- moved MOTOR1 1.42 mm to (1.91, -1.91)
- moved D7 1.27 mm to (-65.4, 58.4)
- moved MOTOR2 1.27 mm to (-15.2, -1.91)
- moved D6 0.64 mm to (-65.4, 62.9)
- moved DRK1 0.64 mm to (-57.1, 67.3)
- moved DRK2 0.63 mm to (-57.1, 38.1)
Routing:
- net GND: track 0.00 -> 482.8 mm, vias 0 -> 2
- net LIPO-GND: track 0.00 -> 322.6 mm, vias 0 -> 5
- net LIPO-VDD: track 0.00 -> 273.0 mm, vias 0 -> 3
- net N$42: track 0.00 -> 210.9 mm, vias 0 -> 1
- net 3.3V: track 0.00 -> 191.5 mm, vias 0 -> 3
- net +3.6V: track 0.00 -> 165.1 mm, vias 0 -> 3
- net N$13: track 0.00 -> 143.2 mm, vias 0 -> 2
- net BLCK-M2: track 0.00 -> 141.1 mm
- net N$1: track 0.00 -> 139.9 mm, vias 0 -> 1
- net TX5: track 0.00 -> 136.1 mm, vias 0 -> 2
- net N$2: track 0.00 -> 129.6 mm
- net N$3: track 0.00 -> 125.1 mm, vias 0 -> 2
- net WH_ENC_B: track 0.00 -> 124.2 mm, vias 0 -> 2
- net RED-M1: track 0.00 -> 119.2 mm
- net SCL1: track 0.00 -> 107.6 mm
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
Commit message: Ordered PCB by Aisler!
Parts:
- moved MOTOR1 0.64 mm to (2.54, -1.91), turned to 270 degrees
- moved ENC0 0.63 mm to (1.91, 9.53)
- moved ENC1 0.63 mm to (-15.9, 9.53)
- moved ENC2 0.63 mm to (-33.7, 9.53)
- turned MOTOR2 to 270 degrees
- turned MOTOR3 to 270 degrees
Routing:
- net LIPO-GND: track 322.6 -> 248.9 mm, vias 5 -> 7
- net N$13: track 143.2 -> 87.1 mm, vias 2 -> 1
- net LIPO-VDD: track 273.0 -> 223.0 mm, vias 3 -> 7
- net N$42: track 210.9 -> 162.3 mm, vias 1 -> 2
- net GND: track 482.8 -> 440.7 mm, vias 2 -> 3
- net BLCK-M2: track 141.1 -> 117.1 mm
- net N$3: track 125.1 -> 145.2 mm, vias 2 -> 0
- net CS0: track 63.4 -> 80.8 mm, vias 4 -> 5
- net N$15: track 75.2 -> 88.1 mm, vias 3 -> 0
- net SDA1: track 102.4 -> 114.5 mm, vias 1 -> 2
- net N$29: track 65.3 -> 77.2 mm, vias 2 -> 1
- net N$44: track 94.8 -> 83.6 mm, vias 3 -> 2
- net MOSI: track 97.7 -> 86.9 mm, vias 2 -> 1
- net Y_ENC_A: track 68.2 -> 61.4 mm, vias 3 -> 0
- net MISO: track 92.9 -> 99.2 mm
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Other:
- board text added: "+3.3V"
- board text added: "CS0"
- board text added: "CS1"
- board text added: "CS2"
- board text added: "MISO"
- board text added: "MOSI"
- board text added: "SCK"
